File: bblan95xx.sch (EAGLE design)
At the start: 49 parts, among them IC1 LAN9512, IC2 93ST, Q1 25MHz

Commit message: add extra analog capacitor and route VDD33A to free PIN
Signed-off-by: Stephan Baerwolf <stephan@matrixstorm.com>
Parts:
- added C29: .1u, resistor:C-EUC0603K
- added R8: (no value), resistor:R-EU_R0402
Connections:
- new net VBIAS: JPUSBETHERNET.5, R8.1
- net GND: now also C29.1
- net VDD33A: now also C29.2, R8.2
Changed lines of the file:
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@@
 <part name="R2" library="resistor" deviceset="R-EU_" device="R0603"/>
 <part name="R1" library="resistor" deviceset="R-EU_" device="R0603"/>
+<part name="C29" library="resistor" deviceset="C-EU" device="C0603K" value=".1u"/>
+<part name="R8" library="resistor" deviceset="R-EU_" device="R0402"/>
 </parts>
 <sheets>
@@
 <instance part="R2" gate="G$1" x="-193.04" y="63.5" rot="R90"/>
 <instance part="R1" gate="G$1" x="-198.12" y="63.5" rot="R90"/>
+<instance part="C29" gate="G$1" x="-205.74" y="73.66" rot="R90"/>
+<instance part="R8" gate="G$1" x="-149.86" y="73.66" rot="R180"/>
 </instances>
 <busses>
@@
 <junction x="-187.96" y="86.36"/>
 <pinref part="L1" gate="G$1" pin="1"/>
-<wire x1="-187.96" y1="86.36" x2="-187.96" y2="71.12" width="0.1524" layer="91"/>
+<wire x1="-187.96" y1="86.36" x2="-187.96" y2="73.66" width="0.1524" layer="91"/>
 <pinref part="R3" gate="G$1" pin="2"/>
 <pinref part="R1" gate="G$1" pin="2"/>
+<wire x1="-187.96" y1="73.66" x2="-187.96" y2="71.12" width="0.1524" layer="91"/>
 <wire x1="-187.96" y1="71.12" x2="-187.96" y2="68.58" width="0.1524" layer="91"/>
 <wire x1="-198.12" y1="68.58" x2="-198.12" y2="71.12" width="0.1524" layer="91"/>
@@
 <junction x="-187.96" y="71.12"/>
 <junction x="-182.88" y="71.12"/>
+<wire x1="-187.96" y1="73.66" x2="-200.66" y2="73.66" width="0.1524" layer="91"/>
+<pinref part="C29" gate="G$1" pin="2"/>
+<junction x="-187.96" y="73.66"/>
+<wire x1="-187.96" y1="73.66" x2="-154.94" y2="73.66" width="0.1524" layer="91"/>
+<pinref part="R8" gate="G$1" pin="2"/>
 </segment>
 </net>
@@
 <wire x1="-213.36" y1="91.44" x2="-213.36" y2="86.36" width="0.1524" layer="91"/>
 <wire x1="-213.36" y1="86.36" x2="-213.36" y2="78.74" width="0.1524" layer="91"/>
-<wire x1="-213.36" y1="78.74" x2="-213.36" y2="71.12" width="0.1524" layer="91"/>
+<wire x1="-213.36" y1="78.74" x2="-213.36" y2="73.66" width="0.1524" layer="91"/>
+<wire x1="-213.36" y1="73.66" x2="-213.36" y2="71.12" width="0.1524" layer="91"/>
 <wire x1="-200.66" y1="142.24" x2="-213.36" y2="142.24" width="0.1524" layer="91"/>
 <pinref part="C3" gate="G$1" pin="1"/>
@@
 <wire x1="-180.34" y1="78.74" x2="-213.36" y2="78.74" width="0.1524" layer="91"/>
 <pinref part="GND1" gate="1" pin="GND"/>
+<pinref part="C29" gate="G$1" pin="1"/>
+<wire x1="-208.28" y1="73.66" x2="-213.36" y2="73.66" width="0.1524" layer="91"/>
+<junction x="-213.36" y="73.66"/>
 </segment>
 <segment>
@@
 </segment>
 </net>
+<net name="VBIAS" class="0">
+<segment>
+<pinref part="R8" gate="G$1" pin="1"/>
+<wire x1="-144.78" y1="73.66" x2="-114.3" y2="73.66" width="0.1524" layer="91"/>
+<label x="-114.3" y="73.66" size="1.778" layer="95" xref="yes"/>
+</segment>
+<segment>
+<pinref part="JPUSBETHERNET" gate="A" pin="5"/>
+<wire x1="162.56" y1="48.26" x2="154.94" y2="48.26" width="0.1524" layer="91"/>
+<label x="154.94" y="48.26" size="1.778" layer="95" rot="R180" xref="yes"/>
+</segment>
+</net>

Commit message: add extra 0603 cap and make 0603 to 0805 where possible
Signed-off-by: Stephan Baerwolf <stephan@matrixstorm.com>
Parts:
- added C30: .1u, resistor:C-EUC0603K
- C1, C12, C2, C26, C27, C3, C4, C5, C6, C7, C8: device resistor:C-EUC0603K -> resistor:C-EUC0805K
Connections:
- net GND: now also C30.1
- net VDD33A: now also C30.2
Changed lines of the file:
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@@
 <part name="GND1" library="supply1" deviceset="GND" device=""/>
 <part name="L1" library="resistor" deviceset="R-EU_" device="R0805" value="120Rat100MHz"/>
-<part name="C1" library="resistor" deviceset="C-EU" device="C0603K" value=".1u"/>
-<part name="C2" library="resistor" deviceset="C-EU" device="C0603K" value=".1u"/>
-<part name="C3" library="resistor" deviceset="C-EU" device="C0603K" value=".1u"/>
-<part name="C4" library="resistor" deviceset="C-EU" device="C0603K" value=".1u"/>
-<part name="C5" library="resistor" deviceset="C-EU" device="C0603K" value=".1u"/>
-<part name="C6" library="resistor" deviceset="C-EU" device="C0603K" value=".1u"/>
-<part name="C7" library="resistor" deviceset="C-EU" device="C0603K" value=".1u"/>
-<part name="C8" library="resistor" deviceset="C-EU" device="C0603K" value=".1u"/>
+<part name="C1" library="resistor" deviceset="C-EU" device="C0805K" value=".1u"/>
+<part name="C2" library="resistor" deviceset="C-EU" device="C0805K" value=".1u"/>
+<part name="C3" library="resistor" deviceset="C-EU" device="C0805K" value=".1u"/>
+<part name="C4" library="resistor" deviceset="C-EU" device="C0805K" value=".1u"/>
+<part name="C5" library="resistor" deviceset="C-EU" device="C0805K" value=".1u"/>
+<part name="C6" library="resistor" deviceset="C-EU" device="C0805K" value=".1u"/>
+<part name="C7" library="resistor" deviceset="C-EU" device="C0805K" value=".1u"/>
+<part name="C8" library="resistor" deviceset="C-EU" device="C0805K" value=".1u"/>
 <part name="C9" library="resistor" deviceset="C-EU" device="C0603K" value=".1u"/>
 <part name="C10" library="resistor" deviceset="C-EU" device="C0603K" value=".1u"/>
 <part name="C11" library="resistor" deviceset="C-EU" device="C0603K" value=".1u"/>
-<part name="C12" library="resistor" deviceset="C-EU" device="C0603K" value=".1u"/>
+<part name="C12" library="resistor" deviceset="C-EU" device="C0805K" value=".1u"/>
 <part name="C13" library="resistor" deviceset="C-EU" device="C0805K" value="4.7u"/>
 <part name="C14" library="resistor" deviceset="C-EU" device="C0603K" value=".1u"/>
@@
 <part name="GND7" library="supply1" deviceset="GND" device=""/>
 <part name="C25" library="resistor" deviceset="C-EU" device="C0805K" value="1u"/>
-<part name="C26" library="resistor" deviceset="C-EU" device="C0603K" value=".1u"/>
+<part name="C26" library="resistor" deviceset="C-EU" device="C0805K" value=".1u"/>
 <part name="GND8" library="supply1" deviceset="GND" device=""/>
 <part name="H1" library="holes" deviceset="MOUNT-HOLE" device="3.2"/>
@@
 <part name="L3" library="resistor" deviceset="R-EU_" device="R0805" value="120Rat100MHz"/>
 <part name="C19" library="resistor" deviceset="C-EU" device="C0805K" value="1.0u"/>
-<part name="C27" library="resistor" deviceset="C-EU" device="C0603K" value=".1u"/>
+<part name="C27" library="resistor" deviceset="C-EU" device="C0805K" value=".1u"/>
 <part name="C16" library="resistor" deviceset="C-EU" device="C0805K" value="4.7u"/>
 <part name="C28" library="resistor" deviceset="C-EU" device="C0603K" value=".1u"/>
@@
 <part name="C29" library="resistor" deviceset="C-EU" device="C0603K" value=".1u"/>
 <part name="R8" library="resistor" deviceset="R-EU_" device="R0402"/>
+<part name="C30" library="resistor" deviceset="C-EU" device="C0603K" value=".1u"/>
 </parts>
 <sheets>
@@
 <instance part="C29" gate="G$1" x="-205.74" y="73.66" rot="R90"/>
 <instance part="R8" gate="G$1" x="-149.86" y="73.66" rot="R180"/>
+<instance part="C30" gate="G$1" x="-205.74" y="93.98" rot="R90"/>
 </instances>
 <busses>
@@
 <wire x1="-187.96" y1="106.68" x2="-187.96" y2="101.6" width="0.1524" layer="91"/>
 <wire x1="-187.96" y1="101.6" x2="-187.96" y2="96.52" width="0.1524" layer="91"/>
-<wire x1="-187.96" y1="96.52" x2="-187.96" y2="91.44" width="0.1524" layer="91"/>
+<wire x1="-187.96" y1="96.52" x2="-187.96" y2="93.98" width="0.1524" layer="91"/>
+<wire x1="-187.96" y1="93.98" x2="-187.96" y2="91.44" width="0.1524" layer="91"/>
 <wire x1="-187.96" y1="91.44" x2="-187.96" y2="86.36" width="0.1524" layer="91"/>
 <wire x1="-180.34" y1="116.84" x2="-187.96" y2="116.84" width="0.1524" layer="91"/>
@@
 <wire x1="-187.96" y1="73.66" x2="-154.94" y2="73.66" width="0.1524" layer="91"/>
 <pinref part="R8" gate="G$1" pin="2"/>
+<pinref part="C30" gate="G$1" pin="2"/>
+<wire x1="-200.66" y1="93.98" x2="-187.96" y2="93.98" width="0.1524" layer="91"/>
+<junction x="-187.96" y="93.98"/>
 </segment>
 </net>
@@
 <wire x1="-213.36" y1="106.68" x2="-213.36" y2="101.6" width="0.1524" layer="91"/>
 <wire x1="-213.36" y1="101.6" x2="-213.36" y2="96.52" width="0.1524" layer="91"/>
-<wire x1="-213.36" y1="96.52" x2="-213.36" y2="91.44" width="0.1524" layer="91"/>
+<wire x1="-213.36" y1="96.52" x2="-213.36" y2="93.98" width="0.1524" layer="91"/>
+<wire x1="-213.36" y1="93.98" x2="-213.36" y2="91.44" width="0.1524" layer="91"/>
 <wire x1="-213.36" y1="91.44" x2="-213.36" y2="86.36" width="0.1524" layer="91"/>
 <wire x1="-213.36" y1="86.36" x2="-213.36" y2="78.74" width="0.1524" layer="91"/>
@@
 <wire x1="-208.28" y1="73.66" x2="-213.36" y2="73.66" width="0.1524" layer="91"/>
 <junction x="-213.36" y="73.66"/>
-</segment>
-<segment>
+<pinref part="C30" gate="G$1" pin="1"/>
+<wire x1="-208.28" y1="93.98" x2="-213.36" y2="93.98" width="0.1524" layer="91"/>
+<junction x="-213.36" y="93.98"/>
+</segment>
+<segment>
